Commit message: model: align sim physics to the real robot (mass + servo torque)
Video of the real robot showed a sprawled, belly-low shuffle, not a clean
trot. Root cause was a sim<->real physics mismatch, not the policy:

- Servo torque: effort 2.0 -> 0.20 N*m and MJCF forcerange now derives from
  params effort (was hardcoded +-2.5). The real servos are MG90S-class micro
  servos (~0.2 N*m stall); sim was ~10x over-torqued. velocity 8 -> 6 rad/s.
- Mass: trunk 1.2 -> 0.5 kg, hip_link 0.10 -> 0.03, shank 0.10 -> 0.015, foot
  0.02 -> 0.005. Total now ~0.7 kg (was ~2.1 kg), matching the measured robot.
- Isaac actuator effort_limit 2.0 -> 0.20, velocity_limit 8 -> 6 to match.

Regenerated URDF/MJCF/servo_map. Verified the model still stands under the
default pose at the realistic torque (settles ~0.052 m, upright 0.99), so it's
both realistic and trainable. Retraining on these params so the learned gait
transfers instead of relying on torque the real servos can't deliver.

Co-Authored-By: Claude Opus 4.8 (1M context) <noreply@anthropic.com>

File: model/robot_dog.urdf (robot description, URDF)
Before this commit: robot robot_dog, 17 links, 16 joints
Links:
- removed link FL_thigh
- removed link FR_thigh
- removed link RL_thigh
- removed link RR_thigh
- link FL_hip_link: mass 0.1 -> 0.03; geometry collision cylinder length=0.05 radius=0.018; visual cylinder length=0.05 radius=0.018
- link FL_shank: mass 0.08 -> 0.015; geometry collision cylinder length=0.13 radius=0.013; visual cylinder length=0.13 radius=0.013
- link FR_hip_link: mass 0.1 -> 0.03; geometry collision cylinder length=0.05 radius=0.018; visual cylinder length=0.05 radius=0.018
- link FR_shank: mass 0.08 -> 0.015; geometry collision cylinder length=0.13 radius=0.013; visual cylinder length=0.13 radius=0.013
- link RL_hip_link: mass 0.1 -> 0.03; geometry collision cylinder length=0.05 radius=0.018; visual cylinder length=0.05 radius=0.018
- link RL_shank: mass 0.08 -> 0.015; geometry collision cylinder length=0.13 radius=0.013; visual cylinder length=0.13 radius=0.013
- link RR_hip_link: mass 0.1 -> 0.03; geometry collision cylinder length=0.05 radius=0.018; visual cylinder length=0.05 radius=0.018
- link RR_shank: mass 0.08 -> 0.015; geometry collision cylinder length=0.13 radius=0.013; visual cylinder length=0.13 radius=0.013
- link base_link: mass 1.2 -> 0.5
Joints:
- removed joint FL_hip
- removed joint FL_thigh
- removed joint FR_hip
- removed joint FR_thigh
- removed joint RL_hip
- removed joint RL_thigh
- removed joint RR_hip
- removed joint RR_thigh
- added joint FL_abd: type revolute, parent base_link, child FL_hip_link, origin xyz=0.12 0.06 0 rpy=0 0 0, axis 1.0 0 0, limit lower=-1.0 upper=1.0 effort=0.2 velocity=6.0
- added joint FR_abd: type revolute, parent base_link, child FR_hip_link, origin xyz=0.12 -0.06 0 rpy=0 0 0, axis -1.0 0 0, limit lower=-1.0 upper=1.0 effort=0.2 velocity=6.0
- added joint RL_abd: type revolute, parent base_link, child RL_hip_link, origin xyz=-0.12 0.06 0 rpy=0 0 0, axis 1.0 0 0, limit lower=-1.0 upper=1.0 effort=0.2 velocity=6.0
- added joint RR_abd: type revolute, parent base_link, child RR_hip_link, origin xyz=-0.12 -0.06 0 rpy=0 0 0, axis -1.0 0 0, limit lower=-1.0 upper=1.0 effort=0.2 velocity=6.0
- joint FL_foot_fixed: origin xyz=0 0 -0.12 rpy=0 0 0 -> xyz=0 0 -0.13 rpy=0 0 0
- joint FL_knee: limit lower=-2.6 upper=-0.2 effort=2.0 velocity=8.0 -> lower=-1.5 upper=1.5 effort=0.2 velocity=6.0; origin xyz=0 0 -0.11 rpy=0 0 0 -> xyz=0 0.05 0 rpy=0 0 0; parent FL_thigh -> FL_hip_link
- joint FR_foot_fixed: origin xyz=0 0 -0.12 rpy=0 0 0 -> xyz=0 0 -0.13 rpy=0 0 0
- joint FR_knee: limit lower=-2.6 upper=-0.2 effort=2.0 velocity=8.0 -> lower=-1.5 upper=1.5 effort=0.2 velocity=6.0; origin xyz=0 0 -0.11 rpy=0 0 0 -> xyz=0 -0.05 0 rpy=0 0 0; parent FR_thigh -> FR_hip_link
- joint RL_foot_fixed: origin xyz=0 0 -0.12 rpy=0 0 0 -> xyz=0 0 -0.13 rpy=0 0 0
- joint RL_knee: limit lower=-2.6 upper=-0.2 effort=2.0 velocity=8.0 -> lower=-1.5 upper=1.5 effort=0.2 velocity=6.0; origin xyz=0 0 -0.11 rpy=0 0 0 -> xyz=0 0.05 0 rpy=0 0 0; parent RL_thigh -> RL_hip_link
- joint RR_foot_fixed: origin xyz=0 0 -0.12 rpy=0 0 0 -> xyz=0 0 -0.13 rpy=0 0 0
- joint RR_knee: limit lower=-2.6 upper=-0.2 effort=2.0 velocity=8.0 -> lower=-1.5 upper=1.5 effort=0.2 velocity=6.0; origin xyz=0 0 -0.11 rpy=0 0 0 -> xyz=0 -0.05 0 rpy=0 0 0; parent RR_thigh -> RR_hip_link
